Commit message: The version corresponding the document

File: rh_gazebo/config/gazebo_realhex_description.urdf.xacro (robot description, xacro)
@@ -14,3 +14,11 @@
         <origin xyz="0.02171 0 0.36" rpy="0 0 0"/>
     </joint>
+    <!-- 加载全局相机 -->
+    <xacro:include filename="$(find rm_description)/urdf/sensors/camera_gazebo.xacro"/>
+    <joint name="head_joint" type="fixed">
+        <parent link="base_link"/>
+        <child link="head_link"/>
+        <origin xyz="0.2 0 0.3" rpy="0 0 0"/>
+    </joint>
+    <xacro:usb_camera prefix="head" type="depth" width="640" height="480" fps="30"/>
 </robot>

Commit message: 0624 实物部署待测版

File: rh_gazebo/config/gazebo_realhex_description.urdf.xacro (robot description, xacro)
@@ -1,18 +1,13 @@
 <?xml version="1.0"?>
 <robot xmlns:xacro="http://www.ros.org/wiki/xacro" name="rh_description">
-    <xacro:arg name="base_link_name" default="rm_base_link"/>
-    <xacro:arg name="fixed_to_world" default="no"/>
     <!-- 包含 rm_gazebo 的 xacro 文件，并传递参数 -->
-    <xacro:include filename="$(find rm_gazebo)/config/gazebo_75_6f_description.urdf.xacro">
-        <xacro:arg name="base_link_name" value="$(arg base_link_name)"/>
-        <xacro:arg name="fixed_to_world" value="$(arg fixed_to_world)"/>
-    </xacro:include>
+    <xacro:include filename="$(find rh_gazebo)/config/arm_75_6f_description.urdf.xacro"/>
     <xacro:include filename="$(find xpkg_urdf_echo_plus)/urdf/sim_base.xacro"/>
     <joint name="arm_base_joint" type="fixed">
-        <parent link="base_link"/>
-        <child link="$(arg base_link_name)"/>
+        <parent link="mobile_base"/>
+        <child link="base_link"/>
         <origin xyz="0.02171 0 0.36" rpy="0 0 0"/>
     </joint>
-    <!-- 加载全局相机 -->
+    <!-- 加载全局相机
     <xacro:include filename="$(find rm_description)/urdf/sensors/camera_gazebo.xacro"/>
     <joint name="head_joint" type="fixed">
@@ -21,4 +16,4 @@
         <origin xyz="0.2 0 0.3" rpy="0 0 0"/>
     </joint>
-    <xacro:usb_camera prefix="head" type="depth" width="640" height="480" fps="30"/>
+    <xacro:usb_camera prefix="head" type="depth" width="640" height="480" fps="30"/> -->
 </robot>
